File: Battery.kicad_pcb (KiCad board)
At the start: 2 copper layers, 30.5 x 29.6 mm, 33 parts, among them J1 C2765186, U1 LGS63030, U2 JNJ-LTAU0106W90/Q15MIL/365-37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, U3 JNJ-LTAU0106W90/Q15MIL/365-37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, U4 JNJ-LTAU0106W90/Q15MIL/365-37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, U5 LM393

Commit message: R1.3
Parts:
- R12: value C17888 -> 0Ω
Connections:
- net Net-(D1-A) renamed SW
- net Net-(U1-OVP) renamed OVP
Routing:
- net 5V: track 59.3 -> 60.1 mm
