File: Battery.kicad_sch (KiCad schematic)
At the start: 29 parts, among them J1 C2765186, U1 LGS63030, U2 JNJ-LTAU0106W90/Q15MIL/365-37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, U3 JNJ-LTAU0106W90/Q15MIL/365-37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, U4 JNJ-LTAU0106W90/Q15MIL/365-37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, U5 LM393

Commit message: R1.3
Parts:
- R12: value C17888 -> 0Ω; Field5 0Ω -> (none); LCSC (none) -> C17888
Connections:
- net SW: now reaches D1.2 (A), L1.2, U1.1 (SW)
- net OVP: now reaches R1.2, R2.1, U1.5 (OVP)
Changed lines of the file:
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@@
+		)
+	)
+	(global_label "SW"
+		(shape input)
+		(at 123.19 34.29 90)
+		(fields_autoplaced yes)
+		(effects
+			(font
+				(size 1.27 1.27)
+			)
+			(justify left)
+		)
+		(property "Intersheetrefs" "${INTERSHEET_REFS}"
+			(at 123.19 28.6439 90)
+			(effects
+				(font
+					(size 1.27 1.27)
+				)
+				(justify left)
+				(hide yes)
+			)
+		)
+	)
+	(global_label "OVP"
+		(shape input)
+		(at 124.46 41.91 90)
+		(fields_autoplaced yes)
+		(effects
+			(font
+				(size 1.27 1.27)
+			)
+			(justify left)
+		)
+		(property "Intersheetrefs" "${INTERSHEET_REFS}"
+			(at 124.46 35.2357 90)
+			(effects
+				(font
+					(size 1.27 1.27)
+				)
+				(justify left)
+				(hide yes)
+			)
 		)
 	)
@@
 			)
 		)
-		(property "Value" "C17888"
-			(at 113.0299 113.03 0)
-			(effects
-				(font
-					(size 1.27 1.27)
-				)
-				(justify left)
-				(hide yes)
+		(property "Value" "0Ω"
+			(at 113.03 115.57 90)
+			(effects
+				(font
+					(size 1.27 1.27)
+				)
+				(justify left)
 			)
 		)
@@
 			)
 		)
-		(property "Field5" "0Ω"
+		(property "LCSC" "C17888"
 			(at 111.76 115.57 90)
 			(effects
@@
 					(size 1.27 1.27)
 				)
+				(hide yes)
 			)
 		)
@@
 			)
 		)
-		(property "Datasheet" ""
+		(property "Datasheet" "https://datasheet.lcsc.com/lcsc/2507261355_Legend-Si-LGS63030B6_C5123976.pdf"
 			(at 111.76 39.37 0)
 			(effects
@@
 			)
 		)
-		(property "Description" ""
+		(property "Description" "https://jlcpcb.com/partdetail/LegendSi-LGS63030B6/C5123976"
 			(at 111.76 39.37 0)
 			(effects
